File: hw/stm32_system_on_module/sdram.kicad_sch (KiCad schematic)
At the start: 9 parts, among them U2 AS4C8M16SA-7TCN

Commit message: HW finished
Parts:
- C20: footprint (none) -> Capacitor_SMD:C_0402_1005Metric
Changed lines of the file:
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@@
 			)
 		)
-		(property "Footprint" ""
+		(property "Footprint" "Capacitor_SMD:C_0402_1005Metric"
 			(at 23.8252 185.42 0)
 			(effects
