File: hw/stm32_system_on_module/stm32_system_on_module.kicad_pcb (KiCad board)
At the start: 8 copper layers, 45 x 46.5 mm, 97 parts, among them J1 Conn_01x02_Pin, J2 DF40C-50DP-0.4V_51_, J3 DF40C-50DP-0.4V_51_, J4 10118192-0002LF, U1 STM32H743ZGT6, U2 AS4C8M16SA-7TCN, U3 AT25FF161A-SSHN-T, U4 CP2102N-A02-GQFN20R, Y1 KC2016Z8.00000C15XXK

Commit message: HW finished
Parts:
- added C1: 4u7, Capacitor_SMD:C_0603_1608Metric, F.Cu at (148.4, 91.3)
- added C2: 1u, Capacitor_SMD:C_0402_1005Metric, F.Cu at (140.9, 105.6)
- added C20: 1u, Capacitor_SMD:C_0402_1005Metric, B.Cu at (126.5, 76.0)
- added C29: 4u7, Capacitor_SMD:C_0603_1608Metric, F.Cu at (120.0, 78.3)
- added C30: 4u7, Capacitor_SMD:C_0603_1608Metric, F.Cu at (118.6, 78.3)
- added H1: MountingHole_Pad, MountingHole:MountingHole_2.2mm_M2_Pad, F.Cu at (150.7, 68.8)
- added SW1: PTS810 SJK 250 SMTR LFS, footprints:PTS810_CNK, F.Cu at (151.4, 83.3)
- added TP1: TestPoint, TestPoint:TestPoint_Pad_D2.0mm, B.Cu at (130.3, 108.5)
- added TP2: TestPoint, TestPoint:TestPoint_Pad_D2.0mm, B.Cu at (135.4, 108.5)
- added TP3: TestPoint, TestPoint:TestPoint_Pad_D2.0mm, B.Cu at (134.2, 100.4)
- added TP4: TestPoint, TestPoint:TestPoint_Pad_D2.0mm, B.Cu at (136.8, 97.7)
- C12, C23, C24, C25, C26, C27, C32, C34, C8, R19, R20, R25, R48, R49, R50: moved to B.Cu
- J1: footprint Connector_PinHeader_2.54mm:PinHeader_1x02_P2.54mm_Vertical -> Connector_PinHeader_2.54mm:PinHeader_1x02_P2.54mm_Vertical_SMD_Pin1Left
- R1, R2: moved to F.Cu
- moved R49 91.0 mm to (114.8, 80.8), turned to 180 degrees
- moved R48 89.7 mm to (114.8, 81.7), turned to 180 degrees
- moved C32 86.9 mm to (120.8, 77.7), turned to -90 degrees
- moved C27 77.9 mm to (129.5, 69.1), turned to -90 degrees
- moved C26 72.8 mm to (134.4, 69.2), turned to -90 degrees
- moved C23 69.0 mm to (132.0, 76.0), turned to 90 degrees
- moved C14 68.8 mm to (117.4, 92.1), turned to 135 degrees
- moved C24 66.1 mm to (136.0, 76.1), turned to 90 degrees
- moved C9 65.5 mm to (116.7, 92.8), turned to 135 degrees
- moved C8 65.0 mm to (120.9, 88.0), turned to 135 degrees
- moved C7 61.9 mm to (125.8, 84.4), turned to 45 degrees
- moved J1 60.5 mm to (150.8, 107.2)
- moved C6 60.3 mm to (128.7, 81.2), turned to 180 degrees
- moved C10 59.4 mm to (121.2, 101.8), turned to -135 degrees
- moved C25 58.0 mm to (146.3, 76.0), turned to 90 degrees
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Connections:
- J2 pad 10: unconnected-(J2-Pad10) -> PC.12
- J2 pad 11: unconnected-(J2-Pad11) -> PG.14
- J2 pad 12: unconnected-(J2-Pad12) -> PD.2
- J2 pad 13: unconnected-(J2-Pad13) -> PB.3
- J2 pad 14: unconnected-(J2-Pad14) -> PD.3
- J2 pad 15: unconnected-(J2-Pad15) -> PB.4
- J2 pad 16: unconnected-(J2-Pad16) -> PD.4
- J2 pad 17: unconnected-(J2-Pad17) -> PB.5
- J2 pad 18: unconnected-(J2-Pad18) -> PD.5
- J2 pad 19: unconnected-(J2-Pad19) -> PB.6
- J2 pad 20: unconnected-(J2-Pad20) -> PG.9
- J2 pad 21: unconnected-(J2-Pad21) -> PB.7
- J2 pad 22: unconnected-(J2-Pad22) -> PD.7
- J2 pad 23: unconnected-(J2-Pad23) -> PB.8
- J2 pad 24: unconnected-(J2-Pad24) -> PD.6
- J2 pad 25: unconnected-(J2-Pad25) -> PB.9
- J2 pad 26: unconnected-(J2-Pad26) -> GND
- J2 pad 27: unconnected-(J2-Pad27) -> PE.3
- J2 pad 28: unconnected-(J2-Pad28) -> GND
- J2 pad 29: unconnected-(J2-Pad29) -> PE.4
- J2 pad 3: unconnected-(J2-Pad3) -> PG.10
- J2 pad 30: unconnected-(J2-Pad30) -> GND
- J2 pad 31: unconnected-(J2-Pad31) -> PE.5
- J2 pad 32: unconnected-(J2-Pad32) -> GND
- J2 pad 33: unconnected-(J2-Pad33) -> PE.6
- J2 pad 34: unconnected-(J2-Pad34) -> GND
- J2 pad 35: unconnected-(J2-Pad35) -> PC.13
- J2 pad 36: unconnected-(J2-Pad36) -> GND
- J2 pad 37: unconnected-(J2-Pad37) -> PC.14
- J2 pad 38: unconnected-(J2-Pad38) -> GND
- J2 pad 39: unconnected-(J2-Pad39) -> PC.15
- J2 pad 4: unconnected-(J2-Pad4) -> PA.15
- J2 pad 40: unconnected-(J2-Pad40) -> GND
- J2 pad 41: unconnected-(J2-Pad41) -> PF.7
- J2 pad 42: unconnected-(J2-Pad42) -> GND
- J2 pad 43: unconnected-(J2-Pad43) -> PC.1
- J2 pad 44: unconnected-(J2-Pad44) -> GND
- J2 pad 45: unconnected-(J2-Pad45) -> GND
- J2 pad 46: unconnected-(J2-Pad46) -> GND
- J2 pad 47: unconnected-(J2-Pad47) -> GND
- J2 pad 48: unconnected-(J2-Pad48) -> GND
- J2 pad 49: unconnected-(J2-Pad49) -> GND
- J2 pad 5: unconnected-(J2-Pad5) -> PG.11
- J2 pad 50: unconnected-(J2-Pad50) -> GND
- J2 pad 6: unconnected-(J2-Pad6) -> PC.10
- J2 pad 7: unconnected-(J2-Pad7) -> PG.12
- J2 pad 8: unconnected-(J2-Pad8) -> PC.11
- J2 pad 9: unconnected-(J2-Pad9) -> PG.13
- J3 pad 1: unconnected-(J3-Pad1) -> PC.9
- J3 pad 10: unconnected-(J3-Pad10) -> GND
- J3 pad 11: unconnected-(J3-Pad11) -> PA.12
- J3 pad 12: unconnected-(J3-Pad12) -> PG.3
- J3 pad 13: unconnected-(J3-Pad13) -> GND
- J3 pad 14: unconnected-(J3-Pad14) -> PG.2
- J3 pad 15: unconnected-(J3-Pad15) -> GND
- J3 pad 16: unconnected-(J3-Pad16) -> PD.13
- J3 pad 17: unconnected-(J3-Pad17) -> GND
- J3 pad 18: unconnected-(J3-Pad18) -> PD.12
- J3 pad 19: unconnected-(J3-Pad19) -> GND
- J3 pad 2: unconnected-(J3-Pad2) -> PC.8
- J3 pad 20: unconnected-(J3-Pad20) -> PD.11
- J3 pad 21: unconnected-(J3-Pad21) -> GND
- J3 pad 22: unconnected-(J3-Pad22) -> PB.13
- J3 pad 23: unconnected-(J3-Pad23) -> GND
- J3 pad 24: unconnected-(J3-Pad24) -> PB.12
- J3 pad 25: unconnected-(J3-Pad25) -> GND
- J3 pad 26: unconnected-(J3-Pad26) -> PB.11
- J3 pad 27: unconnected-(J3-Pad27) -> GND
- J3 pad 28: unconnected-(J3-Pad28) -> PB.2
- J3 pad 29: unconnected-(J3-Pad29) -> GND
- J3 pad 3: unconnected-(J3-Pad3) -> PA.8
- J3 pad 30: unconnected-(J3-Pad30) -> PB.1
- J3 pad 31: unconnected-(J3-Pad31) -> VBUS
- J3 pad 32: unconnected-(J3-Pad32) -> PB.0
- J3 pad 33: unconnected-(J3-Pad33) -> VBUS
- J3 pad 34: unconnected-(J3-Pad34) -> GND
- J3 pad 35: unconnected-(J3-Pad35) -> VBUS
- J3 pad 36: unconnected-(J3-Pad36) -> GND
- J3 pad 37: unconnected-(J3-Pad37) -> VBUS
- J3 pad 38: unconnected-(J3-Pad38) -> PA.7
- J3 pad 39: unconnected-(J3-Pad39) -> VBUS
- J3 pad 4: unconnected-(J3-Pad4) -> PC.7
- J3 pad 40: unconnected-(J3-Pad40) -> PA.6
- J3 pad 41: unconnected-(J3-Pad41) -> VBUS
- J3 pad 42: unconnected-(J3-Pad42) -> PA.5
- J3 pad 43: unconnected-(J3-Pad43) -> VBUS
- J3 pad 44: unconnected-(J3-Pad44) -> PA.4
- J3 pad 45: unconnected-(J3-Pad45) -> VBUS
- J3 pad 46: unconnected-(J3-Pad46) -> GND
- J3 pad 47: unconnected-(J3-Pad47) -> VBUS
- J3 pad 48: unconnected-(J3-Pad48) -> GND
- J3 pad 49: unconnected-(J3-Pad49) -> VBUS
- J3 pad 5: unconnected-(J3-Pad5) -> PA.9
- J3 pad 50: unconnected-(J3-Pad50) -> GND
- J3 pad 6: unconnected-(J3-Pad6) -> GND
- J3 pad 7: unconnected-(J3-Pad7) -> PA.10
- J3 pad 8: unconnected-(J3-Pad8) -> GND
- J3 pad 9: unconnected-(J3-Pad9) -> PA.11
- U1 pad 100: unconnected-(U1A-PA8-Pad100) -> PA.8
- U1 pad 101: unconnected-(U1A-PA9-Pad101) -> PA.9
- U1 pad 102: unconnected-(U1A-PA10-Pad102) -> PA.10
- U1 pad 103: unconnected-(U1A-PA11-Pad103) -> PA.11
- U1 pad 104: unconnected-(U1A-PA12-Pad104) -> PA.12
- U1 pad 105: unconnected-(U1A-PA13-Pad105) -> /MCU/SWD.DIO
- U1 pad 109: unconnected-(U1A-PA14-Pad109) -> /MCU/SWD.CLK
- U1 pad 110: unconnected-(U1A-PA15-Pad110) -> PA.15
- U1 pad 111: unconnected-(U1C-PC10-Pad111) -> PC.10
- U1 pad 112: unconnected-(U1C-PC11-Pad112) -> PC.11
- U1 pad 113: unconnected-(U1C-PC12-Pad113) -> PC.12
- U1 pad 116: unconnected-(U1D-PD2-Pad116) -> PD.2
- U1 pad 117: unconnected-(U1D-PD3-Pad117) -> PD.3
- U1 pad 118: unconnected-(U1D-PD4-Pad118) -> PD.4
- U1 pad 119: unconnected-(U1D-PD5-Pad119) -> PD.5
- U1 pad 122: unconnected-(U1D-PD6-Pad122) -> PD.6
- U1 pad 123: unconnected-(U1D-PD7-Pad123) -> PD.7
- U1 pad 124: unconnected-(U1G-PG9-Pad124) -> PG.9
- U1 pad 125: unconnected-(U1G-PG10-Pad125) -> PG.10
- U1 pad 126: unconnected-(U1G-PG11-Pad126) -> PG.11
- U1 pad 127: unconnected-(U1G-PG12-Pad127) -> PG.12
- U1 pad 128: unconnected-(U1G-PG13-Pad128) -> PG.13
- U1 pad 129: unconnected-(U1G-PG14-Pad129) -> PG.14
- U1 pad 133: unconnected-(U1B-PB3-Pad133) -> PB.3
- U1 pad 134: unconnected-(U1B-PB4-Pad134) -> PB.4
- U1 pad 135: unconnected-(U1B-PB5-Pad135) -> PB.5
- U1 pad 136: unconnected-(U1B-PB6-Pad136) -> PB.6
- U1 pad 137: unconnected-(U1B-PB7-Pad137) -> PB.7
- U1 pad 139: unconnected-(U1B-PB8-Pad139) -> PB.8
- U1 pad 140: unconnected-(U1B-PB9-Pad140) -> PB.9
- U1 pad 19: unconnected-(U1F-PF7-Pad19) -> PF.7
- U1 pad 2: unconnected-(U1E-PE3-Pad2) -> PE.3
- U1 pad 27: unconnected-(U1C-PC1-Pad27) -> PC.1
- U1 pad 3: unconnected-(U1E-PE4-Pad3) -> PE.4
- U1 pad 4: unconnected-(U1E-PE5-Pad4) -> PE.5
- U1 pad 40: unconnected-(U1A-PA4-Pad40) -> PA.4
- U1 pad 41: unconnected-(U1A-PA5-Pad41) -> PA.5
- U1 pad 42: unconnected-(U1A-PA6-Pad42) -> PA.6
- U1 pad 43: unconnected-(U1A-PA7-Pad43) -> PA.7
- U1 pad 46: unconnected-(U1B-PB0-Pad46) -> PB.0
- U1 pad 47: unconnected-(U1B-PB1-Pad47) -> PB.1
- U1 pad 48: unconnected-(U1B-PB2-Pad48) -> PB.2
- U1 pad 5: unconnected-(U1E-PE6-Pad5) -> PE.6
- U1 pad 7: unconnected-(U1C-PC13-Pad7) -> PC.13
- U1 pad 70: unconnected-(U1B-PB11-Pad70) -> PB.11
- U1 pad 73: unconnected-(U1B-PB12-Pad73) -> PB.12
- U1 pad 74: unconnected-(U1B-PB13-Pad74) -> PB.13
- U1 pad 8: unconnected-(U1C-PC14-Pad8) -> PC.14
- U1 pad 80: unconnected-(U1D-PD11-Pad80) -> PD.11
- U1 pad 81: unconnected-(U1D-PD12-Pad81) -> PD.12
- U1 pad 82: unconnected-(U1D-PD13-Pad82) -> PD.13
- U1 pad 87: unconnected-(U1G-PG2-Pad87) -> PG.2
- U1 pad 88: unconnected-(U1G-PG3-Pad88) -> PG.3
- U1 pad 9: unconnected-(U1C-PC15-Pad9) -> PC.15
- U1 pad 97: unconnected-(U1C-PC7-Pad97) -> PC.7
- U1 pad 98: unconnected-(U1C-PC8-Pad98) -> PC.8
- U1 pad 99: unconnected-(U1C-PC9-Pad99) -> PC.9
Routing:
- net GND: track 16.4 -> 179.9 mm, vias 12 -> 42
- net +3V3: track 21.1 -> 78.6 mm, vias 13 -> 37
- net FMC.NBL0: track 0.00 -> 47.9 mm, vias 0 -> 2
- net FMC.BA1: track 0.00 -> 47.8 mm, vias 0 -> 2
- net FMC.SDCKE0: track 0.00 -> 47.8 mm, vias 0 -> 1
- net FMC.BA0: track 0.00 -> 47.6 mm, vias 0 -> 2
- net FMC.A11: track 0.00 -> 47.2 mm, vias 0 -> 2
- net FMC.A5: track 0.00 -> 47.1 mm, vias 0 -> 2
- net FMC.NBL1: track 0.00 -> 47.1 mm, vias 0 -> 2
- net FMC.D14: track 0.00 -> 47.0 mm, vias 0 -> 2
- net FMC.A3: track 0.00 -> 47.0 mm, vias 0 -> 2
- net FMC.D2: track 0.00 -> 47.0 mm, vias 0 -> 2
- net FMC.D3: track 0.00 -> 47.0 mm, vias 0 -> 2
- net FMC.A8: track 0.00 -> 46.9 mm, vias 0 -> 2
- net FMC.SDCLK: track 0.00 -> 46.8 mm, vias 0 -> 2
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- added copper zone on F.Cu, net +3V3
- added copper zone on In3.Cu, net +3V3
- added copper zone on F.Cu, net +5V
- added copper zone on In3.Cu, net +5V
- added copper zone on In4.Cu, net GND
- added copper zone on F.Cu, net LINE
- removed copper zone on In3.Cu, net GND
- removed copper zone on In5.Cu, net GND
Other:
- board size 45 x 46.5 mm -> 44.6 x 46.3 mm
- board text added: "3V3"
- board text added: "BOOT"
- board text added: "CLK"
- board text added: "DIO"
- board text added: "GND"
- board text added: "PWR"
- board text added: "RST"
